File: ProyectoKicad/ProyectoUcurrent/ProyectoUcurrent.kicad_sch (KiCad schematic)
At the start: 14 parts, among them U1 MAX4239AUT, U2 MAX4239AUT, U3 LMV321

Commit message: CreacionPCB_Kicad
Parts:
- removed I1: 500u, symbol Simulation_SPICE:IDC
- removed R1: 9k, symbol Device:R
- removed R4: 1k, symbol Device:R
- removed U3: LMV321, symbol Amplifier_Operational:LMV321
- removed V1: 3, symbol Simulation_SPICE:VDC
- added J1, J2, J3, J4, J5: Conn_01x01_Socket, Connector_Wire:SolderWire-1.5sqmm_1x01_D1.7mm_OD3mm, symbol Connector:Conn_01x01_Socket
- added Q1: BSC028N06LS3, Package_TO_SOT_SMD:TDSON-8-1, symbol Transistor_FET:BSC028N06LS3
- added R10: 10000, Resistor_THT:R_Axial_DIN0414_L11.9mm_D4.5mm_P25.40mm_Horizontal, symbol Device:R
- added R11: 65000, Resistor_THT:R_Axial_DIN0414_L11.9mm_D4.5mm_P25.40mm_Horizontal, symbol Device:R
- added R12: 220, Resistor_THT:R_Axial_DIN0414_L11.9mm_D4.5mm_P25.40mm_Horizontal, symbol Device:R
- added R13: 1k, Resistor_THT:R_Axial_DIN0414_L11.9mm_D4.5mm_P25.40mm_Horizontal, symbol Device:R
- added R14: 9k, Resistor_THT:R_Axial_DIN0414_L11.9mm_D4.5mm_P25.40mm_Horizontal, symbol Device:R
- added R9: 10, Resistor_THT:R_Axial_DIN0414_L11.9mm_D4.5mm_P25.40mm_Horizontal, symbol Device:R
- added U3: 74HC74, Package_DIP:DIP-14_W7.62mm, symbol 74xx:74HC74
- added U5, U6: TLV3501AID, Package_SO:SOIC-8_3.9x4.9mm_P1.27mm, symbol Comparator:TLV3501AID
- added U7: 74AHC2G00, Package_SO:SSOP-8_2.95x2.8mm_P0.65mm, symbol 74xGxx:74AHC2G00
- added U8: LMV321, Package_TO_SOT_SMD:SOT-23-5, symbol Amplifier_Operational:LMV321
- C1: footprint (none) -> Capacitor_SMD:CP_Elec_3x5.3
- R2, R3, R5, R7, R8: footprint (none) -> Resistor_THT:R_Axial_DIN0414_L11.9mm_D4.5mm_P25.40mm_Horizontal
- R6: value 270 -> 50k; footprint (none) -> Resistor_THT:R_Axial_DIN0414_L11.9mm_D4.5mm_P25.40mm_Horizontal
Connections:
- net GNDREF: now also J2.1 (Pin_1), Q1.1 (S), Q1.2 (S), Q1.3 (S), R12.2, R13.2, U5.4 (V-), U5.8 (SHDN), U6.4 (V-), U6.8 (SHDN), U8.3 (-), U8.4
- net V+: now also R10.1, U3.4 (~{S}), U5.7 (V+), U6.7 (V+), U8.5 (V+)
- net V-: now also U8.2 (V-)
- net Vout: now also J3.1 (Pin_1), R14.2; no longer R3.2
- net at R7.1, R8.2: now also U8.1 (+)
- net at R2.2, U1.4 (-): now also R3.1
- net at U1.1, U2.3 (+): now also R3.2
- net Vset: now reaches R6.1, U2.1
- net Vset: now also J4.1 (Pin_1), U5.3 (+), U6.2 (-)
- net at U2.4 (-): now also R13.1, R14.1; no longer R3.1
- net at R5.1, U1.3 (+): now also J1.1 (Pin_1), R9.1
- new net: R11.2, R12.1, U6.3 (+)
- new net: Q1.5 (D), R9.2
- new net: R10.2, R11.1, U5.2 (-)
- new net: U3.2 (D), U5.6
- new net: U6.6, U7.1
- new net: U3.5 (Q), U7.2
- new net: U3.1 (~{R}), U7.7
- new net: J5.1 (Pin_1), U3.3 (C)
Other:
- moved on the sheet: C1, R2, R5, R7, R8, U1, U2
